File: pcb-design/pcb-design.kicad_sch (KiCad schematic)
At the start: 44 parts, among them M1 CSD19502Q5B, Q1 BC846, T1 Transformer_1P_2S, U1 UCC2813D-1

Commit message: Transformer footprint is added.
Parts:
- T1: footprint (none) -> CUSTOM_FOOTPRINTS:Custom_Transformer-P0.5-7
Changed lines of the file:
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@@
     (property "Reference" "T1" (id 0) (at 250.19 33.02 0))
     (property "Value" "Transformer_1P_2S" (id 1) (at 250.19 35.56 0))
-    (property "Footprint" "" (id 2) (at 250.19 48.895 0)
+    (property "Footprint" "CUSTOM_FOOTPRINTS:Custom_Transformer-P0.5-7" (id 2) (at 250.19 48.895 0)
       (effects (font (size 1.27 1.27)) hide)
     )
@@
     )
     (path "/2df7f288-49d1-4fe5-b2e1-78502a8f2d8e"
-      (reference "T1") (unit 1) (value "Transformer_1P_2S") (footprint "")
+      (reference "T1") (unit 1) (value "Transformer_1P_2S") (footprint "CUSTOM_FOOTPRINTS:Custom_Transformer-P0.5-7")
     )
     (path "/7170042a-a2bc-4332-aac4-507f85c08ee1"

Commit message: Schematic is corrected. PCB Design is added.
Parts:
- added H1, H2, H3, H4: MountingHole, MountingHole:MountingHole_3.2mm_M3, symbol Mechanical:MountingHole
Connections:
- net at Cref1.2, O1.4, Qsc1.1 (B2)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: no longer Rt1.1
- net at Dsnub1.2 (A), T1.5 (SC): now also M1.5 (D)
- net at Ct1.1, Qsc1.2 (E), U1.4 (RC): now also Rt1.1
- net at Daux1.1 (K), Raux1.2: no longer M1.5 (D)
Changed lines of the file:
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@@
 (kicad_sch (version 20211123) (generator eeschema)
   (paper "A3")
-  (junction (at 222.25 85.725) (diameter 0) (color 0 0 0 0)
-  )
   (junction (at 59.055 107.315) (diameter 0) (color 0 0 0 0)
   )
   (junction (at 270.51 127.635) (diameter 0) (color 0 0 0 0)
   )
+  (junction (at 35.56 112.395) (diameter 0) (color 0 0 0 0)
+  )
   (junction (at 182.245 85.725) (diameter 0) (color 0 0 0 0)
   )
@@
   (junction (at 177.8 56.515) (diameter 0) (color 0 0 0 0)
   )
+  (junction (at 222.25 56.515) (diameter 0) (color 0 0 0 0)
+  )
   (junction (at 264.795 178.435) (diameter 0) (color 0 0 0 0)
   )
@@
   (junction (at 95.25 135.255) (diameter 0) (color 0 0 0 0)
   )
-  (junction (at 26.035 107.315) (diameter 0) (color 0 0 0 0)
-  )
   (junction (at 80.645 135.255) (diameter 0) (color 0 0 0 0)
   )
@@
     (stroke (width 0) (type default) (color 0 0 0 0))
   )
+  (wire (pts (xy 213.995 71.755) (xy 213.995 59.055))
+    (stroke (width 0) (type default) (color 0 0 0 0))
+  )
   (wire (pts (xy 174.625 102.235) (xy 182.245 102.235))
     (stroke (width 0) (type default) (color 0 0 0 0))
@@
     (stroke (width 0) (type default) (color 0 0 0 0))
   )
-  (wire (pts (xy 222.25 85.725) (xy 203.835 85.725))
-    (stroke (width 0) (type default) (color 0 0 0 0))
-  )
   (wire (pts (xy 59.055 107.315) (xy 93.345 107.315))
     (stroke (width 0) (type default) (color 0 0 0 0))
@@
     (stroke (width 0) (type default) (color 0 0 0 0))
   )
-  (wire (pts (xy 222.25 85.725) (xy 222.25 112.395))
-    (stroke (width 0) (type default) (color 0 0 0 0))
-  )
-  (wire (pts (xy 26.035 107.315) (xy 59.055 107.315))
+  (wire (pts (xy 222.25 56.515) (xy 231.14 56.515))
+    (stroke (width 0) (type default) (color 0 0 0 0))
+  )
+  (wire (pts (xy 222.25 56.515) (xy 222.25 112.395))
     (stroke (width 0) (type default) (color 0 0 0 0))
   )
@@
     (stroke (width 0) (type default) (color 0 0 0 0))
   )
+  (wire (pts (xy 213.995 79.375) (xy 213.995 85.725))
+    (stroke (width 0) (type default) (color 0 0 0 0))
+  )
   (wire (pts (xy 222.25 139.065) (xy 222.25 132.715))
     (stroke (width 0) (type default) (color 0 0 0 0))
@@
     (stroke (width 0) (type default) (color 0 0 0 0))
   )
-  (wire (pts (xy 213.36 56.515) (xy 231.14 56.515))
+  (wire (pts (xy 213.36 56.515) (xy 222.25 56.515))
+    (stroke (width 0) (type default) (color 0 0 0 0))
+  )
+  (wire (pts (xy 213.995 59.055) (xy 240.03 59.055))
     (stroke (width 0) (type default) (color 0 0 0 0))
   )
@@
     (stroke (width 0) (type default) (color 0 0 0 0))
   )
-  (wire (pts (xy 16.51 107.315) (xy 26.035 107.315))
+  (wire (pts (xy 16.51 107.315) (xy 59.055 107.315))
     (stroke (width 0) (type default) (color 0 0 0 0))
   )
@@
     (stroke (width 0) (type default) (color 0 0 0 0))
   )
-  (wire (pts (xy 26.035 133.985) (xy 26.035 107.315))
-    (stroke (width 0) (type default) (color 0 0 0 0))
-  )
   (wire (pts (xy 95.25 140.97) (xy 91.44 140.97))
     (stroke (width 0) (type default) (color 0 0 0 0))
@@
     (stroke (width 0) (type default) (color 0 0 0 0))
   )
+  (wire (pts (xy 26.035 133.985) (xy 26.035 112.395))
+    (stroke (width 0) (type default) (color 0 0 0 0))
+  )
   (wire (pts (xy 102.87 150.495) (xy 144.145 150.495))
     (stroke (width 0) (type default) (color 0 0 0 0))
@@
     (stroke (width 0) (type default) (color 0 0 0 0))
   )
+  (wire (pts (xy 26.035 112.395) (xy 35.56 112.395))
+    (stroke (width 0) (type default) (color 0 0 0 0))
+  )
   (wire (pts (xy 144.145 163.83) (xy 144.145 161.29))
     (stroke (width 0) (type default) (color 0 0 0 0))
@@
     (stroke (width 0) (type default) (color 0 0 0 0))
   )
-  (wire (pts (xy 222.25 80.01) (xy 222.25 85.725))
-    (stroke (width 0) (type default) (color 0 0 0 0))
-  )
-  (wire (pts (xy 222.25 59.055) (xy 222.25 72.39))
+  (wire (pts (xy 213.995 85.725) (xy 203.835 85.725))
     (stroke (width 0) (type default) (color 0 0 0 0))
   )
   (wire (pts (xy 59.055 120.65) (xy 59.055 107.315))
-    (stroke (width 0) (type default) (color 0 0 0 0))
-  )
-  (wire (pts (xy 222.25 59.055) (xy 240.03 59.055))
     (stroke (width 0) (type default) (color 0 0 0 0))
   )
@@
     (pin "1")
     (pin "2")
+  )
+  (symbol (lib_id "Mechanical:MountingHole") (at 43.18 243.205 0) (unit 1)
+    (in_bom yes) (on_board yes) (fields_autoplaced)
+    (property "Reference" "H2" (id 0) (at 45.72 241.9349 0)
+      (effects (font (size 1.27 1.27)) (justify left))
+    )
+    (property "Value" "MountingHole" (id 1) (at 45.72 244.4749 0)
+      (effects (font (size 1.27 1.27)) (justify left))
+    )
+    (property "Footprint" "MountingHole:MountingHole_3.2mm_M3" (id 2) (at 43.18 243.205 0)
+      (effects (font (size 1.27 1.27)) hide)
+    )
+    (property "Datasheet" "~" (id 3) (at 43.18 243.205 0)
+      (effects (font (size 1.27 1.27)) hide)
+    )
   )
   (symbol (lib_id "power:GNDREF") (at 216.535 197.485 0) (unit 1)
@@
     (pin "2")
   )
-  (symbol (lib_id "Device:D_Schottky") (at 222.25 76.2 90) (unit 1)
+  (symbol (lib_name "D_Schottky_1") (lib_id "Device:D_Schottky") (at 213.995 75.565 90) (unit 1)
     (in_bom yes) (on_board yes)
-    (property "Reference" "Daux1" (id 0) (at 224.155 75.565 90)
+    (property "Reference" "Daux1" (id 0) (at 215.9 74.93 90)
       (effects (font (size 1.27 1.27)) (justify right))
     )
-    (property "Value" "D_Schottky" (id 1) (at 224.155 78.105 90)
+    (property "Value" "D_Schottky" (id 1) (at 215.9 77.47 90)
       (effects (font (size 1.27 1.27)) (justify right))
     )
-    (property "Footprint" "Diode_SMD:D_SMA_Handsoldering" (id 2) (at 222.25 76.2 0)
-      (effects (font (size 1.27 1.27)) hide)
-    )
-    (property "Datasheet" "~" (id 3) (at 222.25 76.2 0)
+    (property "Footprint" "Diode_SMD:D_SMA_Handsoldering" (id 2) (at 213.995 75.565 0)
+      (effects (font (size 1.27 1.27)) hide)
+    )
+    (property "Datasheet" "~" (id 3) (at 213.995 75.565 0)
       (effects (font (size 1.27 1.27)) hide)
     )
@@
     (pin "2")
   )
+  (symbol (lib_id "Mechanical:MountingHole") (at 61.595 243.205 0) (unit 1)
+    (in_bom yes) (on_board yes) (fields_autoplaced)
+    (property "Reference" "H4" (id 0) (at 64.135 241.9349 0)
+      (effects (font (size 1.27 1.27)) (justify left))
+    )
+    (property "Value" "MountingHole" (id 1) (at 64.135 244.4749 0)
+      (effects (font (size 1.27 1.27)) (justify left))
+    )
+    (property "Footprint" "MountingHole:MountingHole_3.2mm_M3" (id 2) (at 61.595 243.205 0)
+      (effects (font (size 1.27 1.27)) hide)
+    )
+    (property "Datasheet" "~" (id 3) (at 61.595 243.205 0)
+      (effects (font (size 1.27 1.27)) hide)
+    )
+  )
   (symbol (lib_id "power:VDC") (at 78.74 38.735 90) (unit 1)
     (in_bom yes) (on_board yes) (fields_autoplaced)
@@
     (pin "2")
   )
+  (symbol (lib_id "Mechanical:MountingHole") (at 61.595 235.585 0) (unit 1)
+    (in_bom yes) (on_board yes) (fields_autoplaced)
+    (property "Reference" "H3" (id 0) (at 64.135 234.3149 0)
+      (effects (font (size 1.27 1.27)) (justify left))
+    )
+    (property "Value" "MountingHole" (id 1) (at 64.135 236.8549 0)
+      (effects (font (size 1.27 1.27)) (justify left))
+    )
+    (property "Footprint" "MountingHole:MountingHole_3.2mm_M3" (id 2) (at 61.595 235.585 0)
+      (effects (font (size 1.27 1.27)) hide)
+    )
+    (property "Datasheet" "~" (id 3) (at 61.595 235.585 0)
+      (effects (font (size 1.27 1.27)) hide)
+    )
+  )
+  (symbol (lib_id "Mechanical:MountingHole") (at 43.18 235.585 0) (unit 1)
+    (in_bom yes) (on_board yes) (fields_autoplaced)
+    (property "Reference" "H1" (id 0) (at 45.72 234.3149 0)
+      (effects (font (size 1.27 1.27)) (justify left))
+    )
+    (property "Value" "MountingHole" (id 1) (at 45.72 236.8549 0)
+      (effects (font (size 1.27 1.27)) (justify left))
+    )
+    (property "Footprint" "MountingHole:MountingHole_3.2mm_M3" (id 2) (at 43.18 235.585 0)
+      (effects (font (size 1.27 1.27)) hide)
+    )
+    (property "Datasheet" "~" (id 3) (at 43.18 235.585 0)
+      (effects (font (size 1.27 1.27)) hide)
+    )
+  )
   (symbol (lib_id "Device:C") (at 35.56 125.73 0) (unit 1)
     (in_bom yes) (on_board yes) (fields_autoplaced)
@@
       (reference "Dz1") (unit 1) (value "D_Zener") (footprint "Diode_SMD:D_SOD-123")
     )
+    (path "/f52f1fe1-47ac-436d-90c6-651ed0f814e8"
+      (reference "H1") (unit 1) (value "MountingHole") (footprint "MountingHole:MountingHole_3.2mm_M3")
+    )
+    (path "/518a115a-962b-44c8-a6c2-fc31f93eb9b3"
+      (reference "H2") (unit 1) (value "MountingHole") (footprint "MountingHole:MountingHole_3.2mm_M3")
+    )
+    (path "/f21e2131-c66f-4f0c-baca-360d239c544a"
+      (reference "H3") (unit 1) (value "MountingHole") (footprint "MountingHole:MountingHole_3.2mm_M3")
+    )
+    (path "/c37546b2-9426-4373-94e4-7341703abbff"
+      (reference "H4") (unit 1) (value "MountingHole") (footprint "MountingHole:MountingHole_3.2mm_M3")
+    )
     (path "/c81469bb-3b94-46f2-96c0-a0b2ebc470c7"
